File: SA22C-connector/sa-22c-microsemi-connector-flip.brd (EAGLE design)
At the start: 51.7 x 40.6 mm, 4 parts, among them J1 TMMH-109-01-G-DV-ES-A

Commit message: Final touches before first CAM test.
Routing:
- net VDD15: track 29.6 -> 116.6 mm
- net GND: track 14.1 -> 37.5 mm, vias 10 -> 12
- net N$9: track 39.2 -> 41.9 mm
- net N$7: track 73.6 -> 75.8 mm
- net N$8: track 63.2 -> 64.8 mm
- net N$3: track 67.7 -> 66.5 mm
Changed lines of the file:
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@@
 <wire x1="10.193" y1="18.829" x2="5.08" y2="19.05" width="1.016" layer="1"/>
 <via x="5.08" y="19.05" extent="1-16" drill="0.35"/>
+<via x="6.35" y="19.05" extent="1-16" drill="0.35"/>
+<wire x1="19.05" y1="22.86" x2="13.97" y2="22.86" width="1.016" layer="1"/>
+<wire x1="20.32" y1="21.59" x2="19.304" y2="20.828" width="1.016" layer="1"/>
+<wire x1="19.304" y1="20.828" x2="14.097" y2="20.828" width="1.016" layer="1"/>
+<wire x1="14.097" y1="20.828" x2="16.129" y2="21.209" width="1.016" layer="1"/>
+<wire x1="16.129" y1="21.209" x2="16.129" y2="22.606" width="1.016" layer="1"/>
+<wire x1="16.129" y1="22.606" x2="14.986" y2="21.844" width="1.016" layer="1"/>
+<wire x1="6.731" y1="28.829" x2="7.62" y2="27.94" width="1.016" layer="1"/>
+<wire x1="7.62" y1="27.94" x2="8.636" y2="26.924" width="1.016" layer="1"/>
+<wire x1="8.636" y1="26.924" x2="8.636" y2="28.702" width="1.016" layer="1"/>
+<wire x1="8.636" y1="28.702" x2="6.858" y2="26.924" width="1.016" layer="1"/>
+<via x="7.62" y="27.94" extent="1-16" drill="0.35"/>
 </signal>
 <signal name="N$3">
@@
 <contactref element="JP4" pad="7"/>
 <contactref element="JP1" pad="5"/>
-<wire x1="10.193" y1="24.829" x2="5.08" y2="24.74385" width="0.4064" layer="1"/>
-<wire x1="5.08" y1="24.74385" x2="5.08" y2="30.48" width="0.4064" layer="1"/>
-<wire x1="5.08" y1="30.48" x2="18.4343625" y2="30.48" width="0.4064" layer="1"/>
+<wire x1="18.4343625" y1="30.48" x2="6.35" y2="30.48" width="0.4064" layer="1"/>
 <wire x1="18.4343625" y1="30.48" x2="18.6055625" y2="30.3088" width="0.4064" layer="1"/>
 <wire x1="18.6055625" y1="30.3088" x2="21.2724375" y2="30.3088" width="0.4064" layer="1"/>
@@
 <wire x1="45.72" y1="25.4" x2="44.45" y2="25.4" width="0.4064" layer="1"/>
 <wire x1="44.45" y1="25.4" x2="39.37" y2="25.4" width="0.4064" layer="1"/>
+<wire x1="6.35" y1="30.48" x2="5.08" y2="29.21" width="0.4064" layer="1"/>
+<wire x1="5.08" y1="29.21" x2="5.08" y2="25.4" width="0.4064" layer="1"/>
+<wire x1="5.08" y1="25.4" x2="5.715" y2="24.892" width="0.4064" layer="1"/>
+<wire x1="5.715" y1="24.892" x2="10.193" y2="24.829" width="0.4064" layer="1"/>
 </signal>
 <signal name="N$4">
@@
 <contactref element="JP4" pad="3"/>
 <contactref element="JP1" pad="13"/>
-<wire x1="10.193" y1="16.829" x2="6.35" y2="16.51" width="0.4064" layer="1"/>
-<wire x1="6.35" y1="16.51" x2="6.35" y2="6.35" width="0.4064" layer="1"/>
-<wire x1="6.35" y1="6.35" x2="13.97" y2="6.35" width="0.4064" layer="1"/>
-<wire x1="13.97" y1="6.35" x2="16.51" y2="3.81" width="0.4064" layer="1"/>
-<wire x1="16.51" y1="3.81" x2="44.45" y2="3.81" width="0.4064" layer="1"/>
-<wire x1="44.45" y1="3.81" x2="47.9808" y2="7.3408" width="0.4064" layer="1"/>
+<wire x1="6.35" y1="6.35" x2="12.7" y2="6.35" width="0.4064" layer="1"/>
+<wire x1="12.7" y1="6.35" x2="16.51" y2="2.54" width="0.4064" layer="1"/>
+<wire x1="16.51" y1="2.54" x2="43.18" y2="2.54" width="0.4064" layer="1"/>
+<wire x1="43.18" y1="2.54" x2="47.9808" y2="7.3408" width="0.4064" layer="1"/>
 <wire x1="47.9808" y1="13.97" x2="44.45" y2="15.24" width="0.4064" layer="1"/>
 <wire x1="47.9808" y1="7.3408" x2="47.9808" y2="13.97" width="0.4064" layer="1"/>
 <wire x1="44.45" y1="15.24" x2="39.37" y2="15.24" width="0.4064" layer="1"/>
+<wire x1="6.35" y1="6.35" x2="5.08" y2="7.62" width="0.4064" layer="1"/>
+<wire x1="5.08" y1="7.62" x2="5.08" y2="15.24" width="0.4064" layer="1"/>
+<wire x1="5.08" y1="15.24" x2="6.604" y2="16.764" width="0.4064" layer="1"/>
+<wire x1="6.604" y1="16.764" x2="10.193" y2="16.829" width="0.4064" layer="1"/>
 </signal>
 <signal name="N$8">
@@
 <contactref element="JP4" pad="2"/>
 <contactref element="JP1" pad="15"/>
-<wire x1="10.193" y1="14.829" x2="7.493" y2="14.732" width="0.4064" layer="1"/>
-<wire x1="7.493" y1="14.732" x2="7.62" y2="7.62" width="0.4064" layer="1"/>
-<wire x1="7.62" y1="7.62" x2="15.24" y2="7.62" width="0.4064" layer="1"/>
-<wire x1="15.24" y1="7.62" x2="17.78" y2="5.08" width="0.4064" layer="1"/>
-<wire x1="17.78" y1="5.08" x2="43.18" y2="5.08" width="0.4064" layer="1"/>
-<wire x1="43.18" y1="5.08" x2="46.99" y2="8.89" width="0.4064" layer="1"/>
+<wire x1="8.89" y1="7.62" x2="13.97" y2="7.62" width="0.4064" layer="1"/>
+<wire x1="13.97" y1="7.62" x2="17.78" y2="3.81" width="0.4064" layer="1"/>
+<wire x1="17.78" y1="3.81" x2="41.91" y2="3.81" width="0.4064" layer="1"/>
+<wire x1="41.91" y1="3.81" x2="46.99" y2="8.89" width="0.4064" layer="1"/>
 <wire x1="46.99" y1="8.89" x2="46.99" y2="12.7" width="0.4064" layer="1"/>
 <wire x1="46.99" y1="12.7" x2="44.45" y2="12.7" width="0.4064" layer="1"/>
 <wire x1="44.45" y1="12.7" x2="39.37" y2="12.7" width="0.4064" layer="1"/>
+<wire x1="8.89" y1="7.62" x2="6.35" y2="10.16" width="0.4064" layer="1"/>
+<wire x1="6.35" y1="10.16" x2="6.35" y2="13.97" width="0.4064" layer="1"/>
+<wire x1="6.35" y1="13.97" x2="7.366" y2="14.859" width="0.4064" layer="1"/>
+<wire x1="7.366" y1="14.859" x2="10.193" y2="14.829" width="0.4064" layer="1"/>
 </signal>
 <signal name="N$9">
@@
 <contactref element="JP4" pad="1"/>
 <contactref element="JP1" pad="17"/>
-<wire x1="10.193" y1="12.829" x2="10.193" y2="11.463" width="0.3048" layer="1"/>
-<wire x1="10.193" y1="11.463" x2="10.16" y2="11.43" width="0.3048" layer="1"/>
-<wire x1="10.16" y1="11.43" x2="18.5062" y2="11.43" width="0.3048" layer="1"/>
-<wire x1="18.5062" y1="11.43" x2="18.6266" y2="11.5504" width="0.3048" layer="1"/>
-<wire x1="18.6266" y1="11.5504" x2="21.2514" y2="11.5504" width="0.3048" layer="1"/>
-<wire x1="21.2514" y1="11.5504" x2="21.3718" y2="11.43" width="0.3048" layer="1"/>
-<wire x1="21.3718" y1="11.43" x2="21.59" y2="11.43" width="0.3048" layer="1"/>
-<wire x1="21.59" y1="11.43" x2="25.4" y2="7.62" width="0.3048" layer="1"/>
-<wire x1="25.4" y1="7.62" x2="38.1" y2="7.62" width="0.3048" layer="1"/>
-<wire x1="38.1" y1="7.62" x2="39.37" y2="8.89" width="0.3048" layer="1"/>
+<wire x1="39.37" y1="8.89" x2="35.56" y2="5.08" width="0.3048" layer="1"/>
 <wire x1="39.37" y1="8.89" x2="39.37" y2="10.16" width="0.3048" layer="1"/>
 <wire x1="39.37" y1="10.16" x2="44.45" y2="10.16" width="0.3048" layer="1"/>
+<wire x1="18.7602" y1="5.08" x2="14.9502" y2="8.89" width="0.3048" layer="1"/>
+<wire x1="11.43" y1="8.89" x2="10.16" y2="10.16" width="0.3048" layer="1"/>
+<wire x1="10.16" y1="10.16" x2="10.193" y2="12.829" width="0.3048" layer="1"/>
+<wire x1="35.56" y1="5.08" x2="18.7602" y2="5.08" width="0.3048" layer="1"/>
+<wire x1="14.9502" y1="8.89" x2="11.43" y2="8.89" width="0.3048" layer="1"/>
 </signal>
 <signal name="VDD15">
@@
 <contactref element="JP1" pad="4"/>
 <wire x1="14.547" y1="28.829" x2="14.547" y2="26.829" width="1.016" layer="1"/>
-<wire x1="14.547" y1="28.829" x2="26.543" y2="28.829" width="1.016" layer="1"/>
+<wire x1="14.547" y1="28.829" x2="26.416" y2="28.829" width="1.016" layer="1"/>
+<wire x1="26.416" y1="28.829" x2="26.543" y2="28.829" width="1.016" layer="1"/>
 <wire x1="26.543" y1="28.829" x2="27.94" y2="27.94" width="1.016" layer="1"/>
 <wire x1="27.94" y1="27.94" x2="31.75" y2="27.94" width="1.016" layer="1"/>
-<wire x1="31.75" y1="27.94" x2="31.75" y2="30.48" width="1.016" layer="1"/>
-<wire x1="31.75" y1="30.48" x2="36.83" y2="30.48" width="1.016" layer="1"/>
-<wire x1="36.83" y1="30.48" x2="36.83" y2="27.94" width="1.016" layer="1"/>
+<wire x1="31.75" y1="27.94" x2="31.75" y2="29.21" width="1.016" layer="1"/>
+<wire x1="31.75" y1="29.21" x2="31.75" y2="30.48" width="1.016" layer="1"/>
+<wire x1="31.877" y1="30.48" x2="36.195" y2="30.48" width="1.016" layer="1"/>
+<wire x1="36.195" y1="30.48" x2="36.83" y2="30.48" width="1.016" layer="1"/>
+<wire x1="36.83" y1="30.48" x2="36.83" y2="29.21" width="1.016" layer="1"/>
+<wire x1="36.83" y1="29.21" x2="36.83" y2="27.94" width="1.016" layer="1"/>
+<wire x1="14.478" y1="26.797" x2="27.432" y2="26.797" width="1.016" layer="1"/>
+<wire x1="27.432" y1="26.797" x2="29.21" y2="30.353" width="1.016" layer="1"/>
+<wire x1="29.21" y1="30.353" x2="31.877" y2="30.48" width="1.016" layer="1"/>
+<wire x1="31.75" y1="27.94" x2="15.24" y2="27.94" width="1.016" layer="1"/>
+<wire x1="31.75" y1="27.94" x2="31.242" y2="27.559" width="1.016" layer="1"/>
+<wire x1="31.242" y1="27.559" x2="14.732" y2="27.432" width="1.016" layer="1"/>
+<wire x1="31.75" y1="29.21" x2="26.416" y2="28.829" width="1.016" layer="1"/>
+<wire x1="31.75" y1="30.48" x2="29.464" y2="29.591" width="1.016" layer="1"/>
+<wire x1="31.75" y1="27.94" x2="36.83" y2="27.94" width="1.016" layer="1"/>
+<wire x1="36.83" y1="27.94" x2="31.75" y2="29.21" width="1.016" layer="1"/>
+<wire x1="31.75" y1="29.21" x2="36.83" y2="29.21" width="1.016" layer="1"/>
+<wire x1="36.83" y1="29.21" x2="31.75" y2="30.48" width="1.016" layer="1"/>
+<wire x1="31.75" y1="30.48" x2="31.877" y2="30.48" width="1.016" layer="1"/>
+<wire x1="36.195" y1="30.48" x2="36.195" y2="28.067" width="1.016" layer="1"/>
+<wire x1="31.75" y1="27.94" x2="28.956" y2="28.702" width="1.016" layer="1"/>
 </signal>
 <signal name="VCC5">
@@
 <contactref element="JP5" pad="8"/>
 <contactref element="JP1" pad="16"/>
-<wire x1="14.547" y1="14.829" x2="21.209" y2="14.859" width="1.016" layer="1"/>
-<wire x1="21.209" y1="14.859" x2="24.13" y2="12.7" width="1.016" layer="1"/>
-<wire x1="24.13" y1="12.7" x2="31.75" y2="12.7" width="1.016" layer="1"/>
+<wire x1="22.479" y1="14.859" x2="14.55269375" y2="14.82330625" width="1.016" layer="1"/>
+<wire x1="14.547" y1="14.829" x2="14.55269375" y2="14.82330625" width="1.016" layer="1"/>
+<wire x1="22.479" y1="14.859" x2="25.4" y2="12.7" width="1.016" layer="1"/>
+<wire x1="25.4" y1="12.7" x2="31.75" y2="12.7" width="1.016" layer="1"/>
 <wire x1="31.75" y1="12.7" x2="36.83" y2="12.7" width="1.016" layer="1"/>
 </signal>
