File: GameboyLink/Gameboy-Link-Clock.brd (EAGLE design)
At the start: 67.6 x 39 mm, 38 parts, among them Q1 16MHz, Y1 32.768kHz

Commit message: Ready for final verification before sending to production.
Parts:
- added U$1: (no value), kalshagar-images:PIGMAN1
- added U$2: (no value), kalshagar-images:GB
- moved TP_USB_ID 1.50 mm to (46.5, 5.90)
Routing:
- net N$14: track 5.77 -> 4.23 mm
Other:
- board text added: "GB"
- board text added: "GBLinkClock v1.0 - 2024/03"
- board text added: "PWR SEL"
- board text added: "Select"
- board text added: "USB/Ext"
- board text added: "VUSB"
- board text added: "electrogeek.cc"
Changed lines of the file:
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@@
 <wire x1="15" y1="12" x2="10" y2="12" width="0" layer="20"/>
 <wire x1="10" y1="12" x2="9.4" y2="11.4" width="0" layer="20" curve="90"/>
-<rectangle x1="34.9" y1="27.1" x2="37.8" y2="30" layer="21"/>
-<rectangle x1="47.5" y1="31.7" x2="50.1" y2="34.6" layer="21"/>
-<rectangle x1="21" y1="18.7" x2="24.3" y2="21.4" layer="21"/>
 <text x="55" y="-1" size="1.778" layer="51">+</text>
 <text x="61.3" y="-0.2" size="1.778" layer="51">-</text>
-<text x="17.3" y="23" size="1.778" layer="51" rot="R90">GBO</text>
+<text x="17.3" y="23.7" size="1.778" layer="51" rot="R90">GBO</text>
 <text x="17.4" y="3.1" size="1.778" layer="51" rot="R90">GBA/GBC</text>
+<text x="32" y="2" size="1.778" layer="51">VUSB</text>
+<wire x1="56" y1="26" x2="58" y2="30" width="0.3048" layer="51"/>
+<wire x1="58" y1="30" x2="58" y2="27" width="0.3048" layer="51"/>
+<wire x1="58" y1="27" x2="58" y2="24" width="0.3048" layer="51"/>
+<wire x1="58" y1="24" x2="60" y2="28" width="0.3048" layer="51"/>
+<wire x1="58" y1="27" x2="57" y2="27" width="0.3048" layer="51"/>
+<text x="74.5" y="19.9" size="1.778" layer="51" rot="R90">electrogeek.cc</text>
+<text x="62.9" y="11.2" size="1.016" layer="51">GBLinkClock
+v1.0 - 2024/03</text>
+<wire x1="35.6" y1="30.1" x2="37" y2="30.1" width="0.254" layer="51"/>
+<wire x1="48" y1="11.9" x2="49.2" y2="11.9" width="0.254" layer="51"/>
+<text x="50.4" y="7.9" size="0.8128" layer="51">PWR SEL</text>
+<text x="48.8" y="3.6" size="0.6096" layer="51">Select</text>
+<text x="49.6" y="1" size="0.6096" layer="51">GB</text>
+<text x="48" y="6" size="0.6096" layer="51">USB/Ext</text>
 </plain>
 <attributes>
@@
 </element>
 <element name="JP_POWER_SRC" library="jumper" library_urn="urn:adsk.eagle:library:252" package="JP2" package3d_urn="urn:adsk.eagle:package:15452/1" value="" x="52.77" y="3.79" smashed="yes" rot="R90">
-<attribute name="NAME" x="50.919" y="0.434" size="0.6096" layer="25" ratio="10" rot="R90"/>
 <attribute name="POPULARITY" value="34" x="115" y="33" size="1.778" layer="27" rot="R90" display="off"/>
 <attribute name="VALUE" x="57.088" y="0.234" size="1.27" layer="27" ratio="10" rot="R90"/>
 </element>
 <element name="J_EXT" library="SparkFun-Connectors" package="1X03" value="455-1750-1-ND" x="36.31" y="28.36" smashed="yes" rot="R270">
-<attribute name="NAME" x="37.33" y="30.693" size="0.6096" layer="25" font="vector" ratio="20" rot="R180"/>
+<attribute name="NAME" x="37.907" y="29.63" size="0.6096" layer="25" font="vector" ratio="20" rot="R270"/>
 <attribute name="PROD_ID" value="XXX-00000" x="36.31" y="28.36" size="1.778" layer="27" rot="R270" display="off"/>
 <attribute name="VALUE" value="455-1750-1-ND" x="34.278" y="29.63" size="0.6096" layer="27" font="vector" ratio="20" rot="R270"/>
@@
 <attribute name="VALUE" x="31.69" y="27.23" size="1.27" layer="27" rot="R180"/>
 </element>
-<element name="TP_USB_ID" library="SparkFun-Connectors" package="PAD.03X.05" value="TEST-POINT3X5" x="48" y="6" smashed="yes"/>
+<element name="TP_USB_ID" library="SparkFun-Connectors" package="PAD.03X.05" value="TEST-POINT3X5" x="46.5" y="5.9" smashed="yes"/>
 <element name="DS3231" library="kalshagar" package="SO16W" value="DS3231DS3231-SO16W" x="66.21" y="19.06" smashed="yes" rot="R270">
 <attribute name="NAME" x="67.988" y="24.775" size="1.27" layer="25" ratio="10" rot="R270"/>
@@
 </element>
 <element name="USB_MICRO" library="SparkFun-Connectors" package="USB-B-MICRO-SMD_V03" value="USB_MICROB_PLUGCONN-11752" x="43.36" y="0.95" smashed="yes" rot="R90">
-<attribute name="NAME" x="37.391" y="-0.32" size="0.4064" layer="25" rot="R90"/>
 <attribute name="PROD_ID" value="CONN-11752" x="71.3" y="70.8" size="1.778" layer="27" rot="R90" display="off"/>
 <attribute name="VALUE" x="37.899" y="-0.32" size="0.4064" layer="27" rot="R90"/>
 </element>
 <element name="USB_MINI" library="SparkFun-Connectors" package="USB-MINIB" value="USBSMD" x="26.39" y="4.82" smashed="yes" rot="R90">
-<attribute name="NAME" x="25.12" y="1.01" size="0.4064" layer="25" rot="R90"/>
 <attribute name="PROD_ID" value="CONN-08193" x="68.3" y="22.6" size="1.778" layer="27" rot="R90" display="off"/>
 <attribute name="VALUE" x="26.39" y="1.01" size="0.4064" layer="27" rot="R90"/>
@@
 <attribute name="VALUE" x="50.632" y="12.33" size="0.6096" layer="27" font="vector" ratio="20" rot="R90"/>
 </element>
+<element name="U$1" library="kalshagar-images" package="PIGMAN1" value="" x="19.3" y="30" smashed="yes"/>
+<element name="U$2" library="kalshagar-images" package="GB" value="" x="30.7" y="14.4" smashed="yes"/>
 </elements>
 <signals>
@@
 <wire x1="44.01" y1="3.65" x2="44" y2="3.66" width="0.1524" layer="1"/>
 <wire x1="44" y1="3.66" x2="44" y2="5" width="0.1524" layer="1"/>
-<wire x1="44" y1="5" x2="45" y2="6" width="0.1524" layer="1"/>
-<wire x1="45" y1="6" x2="48" y2="6" width="0.1524" layer="1"/>
+<wire x1="44" y1="5" x2="44.9" y2="5.9" width="0.1524" layer="1"/>
+<wire x1="44.9" y1="5.9" x2="46.5" y2="5.9" width="0.1524" layer="1"/>
 </signal>
 <signal name="USB_VCC">
