File: ResistorCalculator/ResistorCalculator.kicad_pcb (KiCad board)
At the start: 2 copper layers, 50 x 100 mm, 18 parts, among them SW1 SW_SPDT, SW10 SW_SPST, SW11 SW_SPST, SW12 SW_SPST, SW13 SW_SPST, SW2 SW_SPST, SW3 SW_SPST, SW4 SW_SPST, SW5 SW_SPST, SW6 SW_SPST, SW7 SW_SPST, SW8 SW_SPST, SW9 SW_SPST

Commit message: Ready for home production
Connections:
- net Net-(J_Power_In1-Pin_1) renamed GND
Routing:
- added copper zone on B.Cu, net GND
Other:
- board text added: "Gnd"
- board text added: "In"
- board text added: "Out"
- board text added: "Resistor Calculator"
- board text added: "Vcc"
Changed lines of the file:
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@@
 	)
 	(net 0 "")
-	(net 1 "Net-(J_Power_In1-Pin_1)")
+	(net 1 "GND")
 	(net 2 "Net-(J_Power_Out1-Pin_2)")
 	(net 3 "Net-(J_Power_In1-Pin_2)")
@@
 			(layers "*.Cu" "*.Mask")
 			(remove_unused_layers no)
-			(net 1 "Net-(J_Power_In1-Pin_1)")
+			(net 1 "GND")
 			(pinfunction "Pin_1")
 			(pintype "passive")
@@
 			(layers "*.Cu" "*.Mask")
 			(remove_unused_layers no)
-			(net 1 "Net-(J_Power_In1-Pin_1)")
+			(net 1 "GND")
 			(pinfunction "Pin_1")
 			(pintype "passive")
@@
 		(tags "CP Radial series Radial pin pitch 2.50mm  diameter 5mm Electrolytic Capacitor")
 		(property "Reference" "C2"
-			(at -3 -2.5 90)
+			(at -2.5 -2.5 90)
 			(layer "F.SilkS")
 			(effects
@@
 		)
 		(fp_text user "${REFERENCE}"
-			(at -3.5 1.5 90)
+			(at -3 1.5 90)
 			(layer "F.Fab")
 			(effects
@@
 			(layers "*.Cu" "*.Mask")
 			(remove_unused_layers no)
-			(net 1 "Net-(J_Power_In1-Pin_1)")
+			(net 1 "GND")
 			(pintype "passive")
 		)
@@
 			(net 7 "unconnected-(SW1-C-Pad3)")
 			(pinfunction "C")
-			(pintype "passive")
+			(pintype "passive+no_connect")
 		)
 		(model "${KICAD8_3DMODEL_DIR}/Button_Switch_THT.3dshapes/SW_Slide-03_Wuerth-WS-SLTV_10x2.5x6.4_P2.54mm.wrl"
@@
 			(layers "*.Cu" "*.Mask")
 			(remove_unused_layers no)
-			(net 1 "Net-(J_Power_In1-Pin_1)")
+			(net 1 "GND")
 			(pintype "passive")
 		)
@@
 	)
 	(gr_line
+		(start 211 36.5)
+		(end 209 34.5)
+		(stroke
+			(width 0.2)
+			(type default)
+		)
+		(layer "B.Cu")
+	)
+	(gr_line
+		(start 210.5 36)
+		(end 209.5 36)
+		(stroke
+			(width 0.2)
+			(type default)
+		)
+		(layer "B.Cu")
+	)
+	(gr_line
+		(start 209 39)
+		(end 206.5 36.5)
+		(stroke
+			(width 0.2)
+			(type default)
+		)
+		(layer "B.Cu")
+	)
+	(gr_line
+		(start 209 34.5)
+		(end 209 39)
+		(stroke
+			(width 0.2)
+			(type default)
+		)
+		(layer "B.Cu")
+	)
+	(gr_line
 		(start 212.5 28)
 		(end 162.5 28)
@@
 		(layer "Edge.Cuts")
 	)
+	(gr_text "Gnd"
+		(at 184.5 58.5 0)
+		(layer "B.Cu")
+		(effects
+			(font
+				(size 1.5 1.5)
+				(thickness 0.3)
+				(bold yes)
+			)
+			(justify left bottom mirror)
+		)
+	)
+	(gr_text "Resistor Calculator"
+		(at 202 33 0)
+		(layer "B.Cu")
+		(effects
+			(font
+				(size 3 2)
+				(thickness 0.5)
+				(bold yes)
+			)
+			(justify left bottom mirror)
+		)
+	)
+	(gr_text "Out"
+		(at 190 53.5 0)
+		(layer "B.Cu")
+		(effects
+			(font
+				(size 1.5 1.5)
+				(thickness 0.3)
+				(bold yes)
+			)
+			(justify left bottom mirror)
+		)
+	)
+	(gr_text "Vcc"
+		(at 184.5 55.5 0)
+		(layer "B.Cu")
+		(effects
+			(font
+				(size 1.5 1.5)
+				(thickness 0.3)
+				(bold yes)
+			)
+			(justify left bottom mirror)
+		)
+	)
+	(gr_text "In"
+		(at 203.5 53 0)
+		(layer "B.Cu")
+		(effects
+			(font
+				(size 1.5 1.5)
+				(thickness 0.3)
+				(bold yes)
+			)
+			(justify left bottom mirror)
+		)
+	)
 	(segment
 		(start 186.5 57.775)
@@
 		(net 16)
 	)
+	(zone
+		(net 1)
+		(net_name "GND")
+		(layer "B.Cu")
+		(name "GND")
+		(hatch edge 0.5)
+		(connect_pads yes
+			(clearance 0.5)
+		)
+		(min_thickness 0.25)
+		(filled_areas_thickness no)
+		(fill yes
+			(thermal_gap 0.5)
+			(thermal_bridge_width 0.5)
+			(island_removal_mode 1)
+			(island_area_min 10)
+		)
+		(polygon
+			(pts
+				(xy 212.5 62) (xy 201 62) (xy 200.5 61.5) (xy 200.5 57) (xy 205.5 57) (xy 208 59.5) (xy 210.5 59.5)
+				(xy 211 59) (xy 211 50.5) (xy 210.5 50) (xy 207.5 50) (xy 207.5 46) (xy 212.5 46)
+			)
+		)
+	)
 )
