File: ResistorCalculator/ResistorCalculator.kicad_sch (KiCad schematic)
At the start: 18 parts, among them SW1 SW_SPDT, SW10 SW_SPST, SW11 SW_SPST, SW12 SW_SPST, SW13 SW_SPST, SW2 SW_SPST, SW3 SW_SPST, SW4 SW_SPST, SW5 SW_SPST, SW6 SW_SPST, SW7 SW_SPST, SW8 SW_SPST, SW9 SW_SPST

Commit message: Ready for home production
Changed lines of the file:
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@@
+	(wire
+		(pts
+			(xy 60.96 49.53) (xy 60.96 45.72)
+		)
+		(stroke
+			(width 0)
+			(type default)
+		)
+	)
 	(wire
 		(pts
@@
 	(wire
 		(pts
-			(xy 60.96 45.72) (xy 60.96 49.53)
-		)
-		(stroke
-			(width 0)
-			(type default)
-		)
-	)
-	(wire
-		(pts
 			(xy 120.65 109.22) (xy 120.65 106.68)
 		)
@@
 	)
 	(label "GND"
-		(at 55.88 45.72 0)
+		(at 60.96 49.53 0)
 		(fields_autoplaced yes)
 		(effects
