File: Rapide861/Rapide861.kicad_pcb (KiCad board)
At the start: 2 copper layers, 49.5 x 59.5 mm, 10 parts, among them J1 AVR-ISP-6, J2 Conn_02x02_Counter_Clockwise, J3 PORTA, J4 PORTB, J5 Conn_01x02, J6 Conn_01x02, U1 ATtiny861-20P, Y1 12MHz

Commit message: FIX now wired the board properly, generated all the gerbl files too and image in case
Connections:
- J3 pad 1: /MOSI -> Net-(J3-Pin_1)
- J3 pad 2: /MISO -> Net-(J3-Pin_2)
- J3 pad 3: /SCK -> Net-(J3-Pin_3)
- J4 pad 1: Net-(J4-Pin_1) -> /MOSI
- J4 pad 2: Net-(J4-Pin_2) -> /MISO
- J4 pad 3: Net-(J4-Pin_3) -> /SCK
- U1 pad 1: Net-(J4-Pin_1) -> /MOSI
- U1 pad 18: /SCK -> Net-(J3-Pin_3)
- U1 pad 19: /MISO -> Net-(J3-Pin_2)
- U1 pad 2: Net-(J4-Pin_2) -> /MISO
- U1 pad 20: /MOSI -> Net-(J3-Pin_1)
- U1 pad 3: Net-(J4-Pin_3) -> /SCK
Routing:
- net /MOSI: track 37.5 -> 57.8 mm, vias 0 -> 2
- net Net-(J4-Pin_3): track 15.0 -> 0.00 mm
- net Net-(J4-Pin_2): track 15.0 -> 0.00 mm
- net Net-(J4-Pin_1): track 15.0 -> 0.00 mm
- net /SCK: track 50.4 -> 35.5 mm, vias 2 -> 0
- net /MISO: track 44.6 -> 32.4 mm, vias 2 -> 0
- net Net-(J3-Pin_2): track 0.00 -> 9.72 mm
- net Net-(J3-Pin_3): track 0.00 -> 9.44 mm
- net Net-(J3-Pin_1): track 0.00 -> 9.44 mm
- net GND: track 128.5 -> 126.4 mm
